File: power_strip_monitor/power_strip_monitor_reduced.sch (EAGLE design)
At the start: 72 parts, among them Q1 4.096MHz, U1 CS5467, U2 CS5467, U4 ATMEGA168, U5 RAC01_02-SC, U6 XBEE-1B1

Commit message: Added LEDs on schematic and layout
Parts:
- added LED1, LED2: (no value), led:LEDCHIPLED_0805
Connections:
- new net N$1: LED2.A, U4.PB1(OC1A)
- new net N$3: LED1.A, U4.PB2(SS/OC1B)
- net GND: now also LED1.C, LED2.C
Changed lines of the file:
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@@
 <?xml version="1.0" encoding="utf-8"?>
 <!DOCTYPE eagle SYSTEM "eagle.dtd">
-<eagle version="6.1">
+<eagle version="6.2">
 <drawing>
 <settings>
@@
 <part name="N3" library="Cool_Electricity" deviceset="1P_HOLE" device=""/>
 <part name="N4" library="Cool_Electricity" deviceset="1P_HOLE" device=""/>
+<part name="LED1" library="led" deviceset="LED" device="CHIPLED_0805"/>
+<part name="LED2" library="led" deviceset="LED" device="CHIPLED_0805"/>
+<part name="GND5" library="SparkFun" deviceset="GND" device=""/>
 </parts>
 <sheets>
@@
 <instance part="N3" gate="G$1" x="-99.06" y="180.34"/>
 <instance part="N4" gate="G$1" x="-96.52" y="142.24"/>
+<instance part="LED1" gate="G$1" x="353.06" y="165.1"/>
+<instance part="LED2" gate="G$1" x="363.22" y="165.1"/>
+<instance part="GND5" gate="1" x="358.14" y="154.94"/>
 </instances>
 <busses>
@@
 <wire x1="317.5" y1="109.22" x2="327.66" y2="109.22" width="0.1524" layer="91"/>
 <wire x1="327.66" y1="109.22" x2="327.66" y2="104.14" width="0.1524" layer="91"/>
+</segment>
+<segment>
+<pinref part="LED1" gate="G$1" pin="C"/>
+<pinref part="GND5" gate="1" pin="GND"/>
+<wire x1="353.06" y1="160.02" x2="358.14" y2="160.02" width="0.1524" layer="91"/>
+<wire x1="358.14" y1="160.02" x2="358.14" y2="157.48" width="0.1524" layer="91"/>
+<pinref part="LED2" gate="G$1" pin="C"/>
+<wire x1="358.14" y1="160.02" x2="363.22" y2="160.02" width="0.1524" layer="91"/>
+<junction x="358.14" y="160.02"/>
 </segment>
 </net>
@@
 </segment>
 </net>
+<net name="N$1" class="0">
+<segment>
+<pinref part="U4" gate="G$1" pin="PB1(OC1A)"/>
+<pinref part="LED2" gate="G$1" pin="A"/>
+<wire x1="320.04" y1="172.72" x2="363.22" y2="172.72" width="0.1524" layer="91"/>
+<wire x1="363.22" y1="172.72" x2="363.22" y2="167.64" width="0.1524" layer="91"/>
+</segment>
+</net>
+<net name="N$3" class="0">
+<segment>
+<pinref part="U4" gate="G$1" pin="PB2(SS/OC1B)"/>
+<pinref part="LED1" gate="G$1" pin="A"/>
+<wire x1="320.04" y1="170.18" x2="353.06" y2="170.18" width="0.1524" layer="91"/>
+<wire x1="353.06" y1="170.18" x2="353.06" y2="167.64" width="0.1524" layer="91"/>
+</segment>
+</net>

Commit message: Added DRC rules, second LINE hole
Parts:
- added LINE1: 1P_HOLE, Cool_Electricity:1P_HOLE
Connections:
- net HOT: now also LINE1.1
Changed lines of the file:
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@@
 <?xml version="1.0" encoding="utf-8"?>
 <!DOCTYPE eagle SYSTEM "eagle.dtd">
-<eagle version="6.2">
+<eagle version="6.1">
 <drawing>
 <settings>
@@
 <part name="LED2" library="led" deviceset="LED" device="CHIPLED_0805"/>
 <part name="GND5" library="SparkFun" deviceset="GND" device=""/>
+<part name="LINE1" library="Cool_Electricity" deviceset="1P_HOLE" device=""/>
 </parts>
 <sheets>
@@
 <instance part="LED2" gate="G$1" x="363.22" y="165.1"/>
 <instance part="GND5" gate="1" x="358.14" y="154.94"/>
+<instance part="LINE1" gate="G$1" x="43.18" y="317.5"/>
 </instances>
 <busses>
@@
 <wire x1="66.04" y1="317.5" x2="66.04" y2="307.34" width="0.1524" layer="91"/>
 <pinref part="LINE" gate="G$1" pin="1"/>
-<wire x1="55.88" y1="307.34" x2="43.18" y2="307.34" width="0.1524" layer="91"/>
-</segment>
-</net>
+<wire x1="55.88" y1="307.34" x2="50.8" y2="307.34" width="0.1524" layer="91"/>
+<wire x1="50.8" y1="307.34" x2="43.18" y2="307.34" width="0.1524" layer="91"/>
+<wire x1="50.8" y1="307.34" x2="50.8" y2="317.5" width="0.1524" layer="91"/>
+<junction x="50.8" y="307.34"/>
+<pinref part="LINE1" gate="G$1" pin="1"/>
+<wire x1="50.8" y1="317.5" x2="43.18" y2="317.5" width="0.1524" layer="91"/>
+</segment>
+</net>

Commit message: Added plastic mount
Other:
- note added: "AN0"
- note added: "AN1"
- note added: "AN2"
- note added: "AN3"
- note added: "AN4"
- note added: "AN5"
- note added: "DIG0"
- note added: "DIG1"
- note added: "DIG10 (PWM)"
- note added: "DIG11 (PWM)"
- note added: "DIG12"
- note added: "DIG13"
- note added: "DIG14"
- note added: "DIG15"
- note added: "DIG16"
- note added: "DIG17"
- note added: "DIG18"
- note added: "DIG19"
- note added: "DIG2"
- note added: "DIG3"
- note added: "DIG4"
- note added: "DIG5 (PWM)"
- note added: "DIG6 (PWM)"
- note added: "DIG7"
- note added: "DIG8"
- note added: "DIG9 (PWM)"
Changed lines of the file:
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@@
 <text x="-48.26" y="254" size="1.778" layer="97">Wattage: 400mW</text>
 <text x="55.88" y="294.64" size="1.778" layer="97">NOTE: GND=NEUTRAL</text>
+<text x="347.98" y="220.98" size="1.778" layer="97">AN0</text>
+<text x="347.98" y="218.44" size="1.778" layer="97">AN1</text>
+<text x="347.98" y="215.9" size="1.778" layer="97">AN2</text>
+<text x="347.98" y="213.36" size="1.778" layer="97">AN3</text>
+<text x="347.98" y="210.82" size="1.778" layer="97">AN4</text>
+<text x="347.98" y="208.28" size="1.778" layer="97">AN5</text>
+<text x="401.32" y="198.12" size="1.778" layer="97">DIG0</text>
+<text x="401.32" y="195.58" size="1.778" layer="97">DIG1</text>
+<text x="401.32" y="193.04" size="1.778" layer="97">DIG2</text>
+<text x="401.32" y="190.5" size="1.778" layer="97">DIG3</text>
+<text x="401.32" y="187.96" size="1.778" layer="97">DIG4</text>
+<text x="401.32" y="185.42" size="1.778" layer="97">DIG5 (PWM)</text>
+<text x="401.32" y="182.88" size="1.778" layer="97">DIG6 (PWM)</text>
+<text x="401.32" y="180.34" size="1.778" layer="97">DIG7</text>
+<text x="401.32" y="175.26" size="1.778" layer="97">DIG8</text>
+<text x="401.32" y="172.72" size="1.778" layer="97">DIG9 (PWM)</text>
+<text x="401.32" y="170.18" size="1.778" layer="97">DIG10 (PWM)</text>
+<text x="401.32" y="167.64" size="1.778" layer="97">DIG11 (PWM)</text>
+<text x="401.32" y="165.1" size="1.778" layer="97">DIG12</text>
+<text x="401.32" y="162.56" size="1.778" layer="97">DIG13</text>
+<text x="358.14" y="220.98" size="1.778" layer="97">DIG14</text>
+<text x="358.14" y="218.44" size="1.778" layer="97">DIG15</text>
+<text x="358.14" y="215.9" size="1.778" layer="97">DIG16</text>
+<text x="358.14" y="213.36" size="1.778" layer="97">DIG17</text>
+<text x="358.14" y="210.82" size="1.778" layer="97">DIG18</text>
+<text x="358.14" y="208.28" size="1.778" layer="97">DIG19</text>
 </plain>
 <instances>
