File: power_strip_monitor/power_strip_monitor_V2.brd (EAGLE design)
At the start: 100 x 80 mm, 108 parts, among them Q1 4.096MHz, U1 CS5467, U10 LTP5901, U2 CS5467, U3 CS5467, U4 ATMEGA168, U5 LNK302, U6 XBEE-1B1, U8 SN74VC4245A, U9 SN74VC4245A

Commit message: Finished, now optimize
Parts:
- removed C32: 22p, SparkFun:0603
- removed LINE, LINE1, NEUTRAL: 1P_HOLE, Cool_Electricity:14GAUGE_HOLE
- added C30: 22p, SparkFun:0603
- added HOT, NEUT1, NEUT2: 1P_HOLE, Cool_Electricity:14GAUGE_HOLE
- added IC1: 74HC595D, 74xx-eu:SO16
- added Q10, Q11, Q8, Q9: (no value), Cool_Electricity:SOT-563_ON
- added Q2, Q3, Q4, Q5, Q6, Q7: BTA312B-800E, Cool_Electricity:D2PACK_NXP
- added R28, R29: 150, SparkFun:0603
- LED1, LED2: device led:CHIPLED_0805 -> led:CHIP-LED0805
- Q1: value 4.096MHz -> 16.384MHz
- R26: value 10k -> 2k 1%
- R27: value 10k -> 4.06k 1%
- moved LED2 324.2 mm to (-260.4, -133.3)
- moved LED1 323.3 mm to (-254.0, -133.3)
- moved C31 269.2 mm to (-168.9, -109.2)
- moved Q1 197.3 mm to (-166.4, -102.9)
- moved R27 181.1 mm to (15.2, 5.08)
- moved R26 172.3 mm to (7.62, 1.27)
- moved C17 153.7 mm to (10.2, 20.3), turned to 180 degrees
- moved C16 145.6 mm to (10.2, 44.5), turned to 180 degrees
- moved U6 143.5 mm to (85.1, 6.35)
- moved C18 129.1 mm to (12.7, 7.62), turned to 90 degrees
- moved R25 124.2 mm to (2.54, 66.0), turned to 270 degrees
- moved R24 123.3 mm to (99.1, 80.0)
- moved L1 120.1 mm to (3.81, 31.8), turned to 270 degrees
- moved D1 118.2 mm to (2.54, 53.3), turned to 270 degrees
- moved U10 110.5 mm to (81.3, 21.6)
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- renumbered N1 to H1, N2 to H2, N3 to H3, N4 to H4, N5 to H5, N6 to H6
Connections:
- removed net HOT: LINE.P$1, LINE1.P$1, R19.2, R25.P$1
- removed net NRET1: H1.P$1, R1.2, R2.2
- removed net NRET2: H2.P$1, R4.2, R5.2
- removed net NRET3: H3.P$1, R7.2, R8.2
- removed net NRET4: H4.P$1, R10.2, R11.2
- removed net NRET5: H5.P$1, R13.2, R14.2
- removed net NRET6: H6.P$1, R16.2, R17.2
- new net GATE1: Q2.3, Q8.1
- new net GATE2: Q3.3, Q8.4
- new net GATE3: Q4.3, Q9.1
- new net GATE4: Q5.3, Q9.4
- new net GATE5: Q10.1, Q6.3
- new net GATE6: Q10.4, Q7.3
- new net HRET1: Q2.1, R1.2, R2.2
- new net HRET2: Q3.1, R4.2, R5.2
- new net HRET3: Q4.1, R7.2, R8.2
- new net HRET4: Q5.1, R10.2, R11.2
- new net HRET5: Q6.1, R13.2, R14.2
- new net HRET6: Q7.1, R16.2, R17.2
- new net LATCH_CLK: IC1.11, U4.32
- new net LATCH_DAT: IC1.14, U4.12
- new net LATCH_LAT: IC1.12, U4.14
- new net LED1: IC1.15, Q11.5
- new net LED2: IC1.7, Q11.2
- new net N$18: H2.P$1, Q3.2
- new net N$19: IC1.3, Q9.2
- new net N$20: H3.P$1, Q4.2
- new net N$21: H4.P$1, Q5.2
- new net N$22: IC1.4, Q9.5
- new net N$23: H5.P$1, Q6.2
- new net N$24: IC1.5, Q10.2
- new net N$25: H6.P$1, Q7.2
- new net N$26: IC1.6, Q10.5
- new net N$28: LED1.A, Q11.4
- new net N$29: LED2.A, Q11.1
- new net N$30: LED2.C, R29.2
- new net N$31: LED1.C, R28.2
- new net N$9: H1.P$1, Q2.2
- new net NEUTRAL: NEUT1.P$1, NEUT2.P$1, R19.2, R25.P$1
- net 5V: now also IC1.10, IC1.16, Q10.3, Q10.6, Q11.3, Q11.6, Q8.3, Q8.6, Q9.3, Q9.6
- net GND: now also C30.2, HOT.P$1, IC1.13, IC1.8, R28.1, R29.1; no longer C32.2, LED1.C, LED2.C, NEUTRAL.P$1
- net N$1: now also C30.1, Q1.2, U4.7; no longer LED2.A, U4.13
- net N$16: now also IC1.1, Q8.2; no longer C31.1, Q1.2, U4.7
- net N$17: now also IC1.2, Q8.5; no longer C32.1, Q1.1, U4.8
- net N$3: now also C31.1, Q1.1, U4.8; no longer LED1.A, U4.14
- net XIN: now also U4.13; no longer U4.12

Commit message: components placed
Parts:
- removed C10, C11, C12, C4, C5, C6, C7, C8, C9: 10n, SparkFun:0603
- removed C16, C17: 4.7uF 400V, SparkFun-Passives:CPOL-RADIAL-1000UF-63V
- removed C18: 100n, SparkFun:0603
- removed C22: 10u 35V, SparkFun-Capacitors:1206
- removed D1: S1M-13-F, Cool_Electricity:SMA-DIODE-KIT
- removed D2, D3: ES1D, Cool_Electricity:SMA-DIODE-KIT
- removed L1: ELL-6UH102M, Cool_Electricity:ELL6RH
- removed L2: PM5022-102M-RC, Cool_Electricity:PM5022
- removed R11, R12, R14, R15, R17, R18, R8, R9: 330 1%, SparkFun:0603
- removed R22, R23, R24, R46: 10k, SparkFun:0603
- removed R26: 2k 1%, SparkFun:0603
- removed R27: 4.06k 1%, SparkFun:0603
- removed TP1, TP10, TP11, TP12, TP18, TP2, TP3, TP4, TP5, TP6, TP7, TP8, TP9: TESTPOINTSMALLEST, WSNlib:TESTPOINT
- C1, C2, C3: value 10n -> CAP_ARRAY; device SparkFun:0603 -> Cool_Electricity:1206_NETWORK
- R2, R3, R5: value 330 1% -> 220 1%; device SparkFun:0603 -> Cool_Electricity:1206_NETWORK
- R25: value FKN200JR-73-8R2 -> S14K680; device SparkFun-Resistors:AXIAL-0.6 -> varistor:S14K680
- R6: value 330 1% -> (none); device SparkFun:0603 -> Cool_Electricity:1206_NETWORK
- U5: value LNK302 -> RAC01_02-SC; device Cool_Electricity:SO-8C_POWERINT -> Cool_Electricity:RAC01_02-SC
- moved R29 412.2 mm to (85.0, 77.0), turned to 180 degrees
- moved R28 409.1 mm to (85.0, 75.0), turned to 180 degrees
- moved LED2 401.0 mm to (81.0, 77.0), turned to 270 degrees
- moved Q11 397.8 mm to (77.5, 70.2), turned to 270 degrees
- moved LED1 394.5 mm to (81.0, 75.0), turned to 270 degrees
- moved Q10 372.5 mm to (69.2, 61.2), turned to 270 degrees
- moved Q9 371.2 mm to (69.2, 63.8), turned to 270 degrees
- moved Q8 369.9 mm to (69.2, 66.2), turned to 270 degrees
- moved Q7 349.5 mm to (59.0, 69.0), flipped to the bottom
- moved Q6 338.5 mm to (59.0, 69.0)
- moved C30 319.2 mm to (90.0, 72.0), turned to 180 degrees
- moved Q5 315.9 mm to (45.0, 69.0), flipped to the bottom
- moved C31 312.8 mm to (86.0, 72.0)
- moved Q1 305.6 mm to (87.6, 67.1)
- moved Q4 305.4 mm to (45.0, 69.0)
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Connections:
- removed net N$10: C22.1, D3.C, R27.1
- removed net N$12: C18.2, U5.1
- removed net N$13: C18.1, C22.2, D2.C, L2.P$1, R26.1, U5.5, U5.6, U5.7, U5.8
- removed net N$14: R26.2, R27.2, U5.2
- removed net N$6: D1.A, R25.P$2
- removed net N$7: C16.1, D1.C, L1.1
- removed net N$8: C17.1, L1.2, U5.4
- net #CS1: now also R6.A1; no longer R24.1
- net #CS2: now also R6.B1; no longer R23.1
- net #CS3: now also R6.C1; no longer R22.1
- net 5V: now also R6.A2, R6.B2, R6.C2, R6.D2, U5.4; no longer D3.A, L2.P$2, R22.2, R23.2, R24.2, R46.2
- net GND: now also C1.A2, C1.B2, C1.C2, C1.D2, C2.A2, C2.B2, C2.C2, C2.D2, C3.A2, C3.B2, C3.C2, C3.D2, R2.B1, R2.D1, R25.1, R3.B1, R3.D1, R5.B1, R5.D1, U5.1, U5.3; no longer C1.2, C10.1, C11.2, C12.1, C16.2, C17.2, C2.1, C3.2, C4.1, C5.2, C6.1, C7.2, C8.1, C9.2, D2.A, R12.2, R15.2, R18.2, R3.2, R6.2, R9.2
- net HRET1: now also R2.A1; no longer R2.2
- net HRET2: now also R2.C1; no longer R5.2
- net HRET3: now also R3.A1; no longer R8.2
- net HRET4: now also R3.C1; no longer R11.2
- net HRET5: now also R5.A1; no longer R14.2
- net HRET6: now also R5.C1; no longer R17.2
- net I1+: now also C1.A1, R2.A2; no longer C1.1, R2.1, TP2.P$1
- net I1-: now also C1.B1, R2.B2; no longer C2.2, R3.1, TP1.P$1
- net I2+: now also C1.C1, R2.C2; no longer C3.1, R5.1, TP3.P$1
- net I2-: now also C1.D1, R2.D2; no longer C4.2, R6.1, TP4.P$1
- net I3+: now also C2.A1, R3.A2; no longer C5.1, R8.1, TP5.P$1
- net I3-: now also C2.B1, R3.B2; no longer C6.2, R9.1, TP6.P$1
- net I4+: now also C2.C1, R3.C2; no longer C7.1, R11.1, TP7.P$1
- net I4-: now also C2.D1, R3.D2; no longer C8.2, R12.1, TP8.P$1
- net I5+: now also C3.A1, R5.A2; no longer C9.1, R14.1, TP9.P$1
- net I5-: now also C3.B1, R5.B2; no longer C10.2, R15.1, TP10.P$1
- net I6+: now also C3.C1, R5.C2; no longer C11.1, R17.1, TP11.P$1
- net I6-: now also C3.D1, R5.D2; no longer C12.2, R18.1, TP12.P$1
- net NEUTRAL: now also R25.2, U5.2; no longer R25.P$1
- net RST: now also R6.D1; no longer R46.1
- net V+: no longer TP18.P$1

Commit message: Trying to route now
Parts:
- Q10, Q11, Q8, Q9: device Cool_Electricity:SOT-563_ON -> Cool_Electricity:SO08
- moved IC1 14.3 mm to (88.6, 67.2), flipped to the bottom, turned to 180 degrees
- moved Q10 10.8 mm to (74.0, 71.0), flipped to the bottom
- moved Q8 8.67 mm to (74.0, 59.0), flipped to the bottom
- moved Q11 7.60 mm to (74.0, 77.0), flipped to the bottom
- moved Q9 4.91 mm to (74.0, 65.0), flipped to the bottom
- moved R28 0.25 mm to (85.0, 74.8)
Connections:
- net 5V: now also Q10.1, Q11.1, Q8.1, Q9.1; no longer Q10.6, Q11.6, Q8.6, Q9.6
- net GATE1: now also Q8.7, Q8.8; no longer Q8.1
- net GATE2: now also Q8.5, Q8.6; no longer Q8.4
- net GATE3: now also Q9.7, Q9.8; no longer Q9.1
- net GATE4: now also Q9.5, Q9.6; no longer Q9.4
- net GATE5: now also Q10.7, Q10.8; no longer Q10.1
- net GATE6: now also Q10.5, Q10.6; no longer Q10.4
- net LED1: now also Q11.2; no longer Q11.5
- net LED2: now also Q11.4; no longer Q11.2
- net N$17: now also Q8.4; no longer Q8.5
- net N$22: now also Q9.4; no longer Q9.5
- net N$26: now also Q10.4; no longer Q10.5
- net N$28: now also Q11.7, Q11.8; no longer Q11.4
- net N$29: now also Q11.5, Q11.6; no longer Q11.1
Routing:
- net GND: track 0.00 -> 618.2 mm, vias 0 -> 3
- net 5V: track 0.00 -> 313.8 mm, vias 0 -> 2
- net #CS1: track 0.00 -> 171.3 mm, vias 0 -> 3
- net 3.3V: track 0.00 -> 117.4 mm
- net SCLK: track 0.00 -> 87.1 mm, vias 0 -> 5
- net MISO: track 0.00 -> 86.0 mm, vias 0 -> 3
- net GATE2: track 0.00 -> 79.3 mm
- net XIN: track 0.00 -> 75.9 mm, vias 0 -> 4
- net MOTE_RESETN_3V: track 0.00 -> 75.3 mm, vias 0 -> 2
- net V+: track 0.00 -> 71.1 mm, vias 0 -> 3
- net MOTE_RX_CTSN_3V: track 0.00 -> 65.5 mm, vias 0 -> 5
- net MOSI: track 0.00 -> 59.9 mm
- net MOTE_TO_ATMEGA_3V: track 0.00 -> 58.7 mm, vias 0 -> 3
- net RST: track 0.00 -> 56.1 mm, vias 0 -> 1
- net V-: track 0.00 -> 55.4 mm, vias 0 -> 5
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
Commit message: Latest Powerstrip changes
Parts:
- removed IC1: 74HC595D, 74xx-eu:SO16
- removed Q10, Q11, Q8, Q9: (no value), Cool_Electricity:SO08
- removed R28, R29: 150, SparkFun:0603
- removed U4: ATMEGA168, SparkFun:TQFP32-08
- removed U6: XBEE-1B1, SparkFun:XBEE-1
- added IC2: ATMEGA644A, atmel:TQFP44
- added J1: EXP, SparkFun-Connectors:2X3
- added R8, R9: 100, Cool_Electricity:1206_NETWORK
- added U$15: XBEE-1B3, SparkFun-RF:XBEE-SMD
- JP2: value AVR_SPI_PRG_6NS -> JTAG; device SparkFun:2X3-NS -> SparkFun-Connectors:AVR_ICSP
- LED1, LED2: device led:CHIP-LED0805 -> led:CHIPLED_0805
- moved H4 84.6 mm to (7.00, 3.00)
- moved H5 81.9 mm to (21.0, 3.00)
- moved H6 78.8 mm to (35.0, 3.00)
- moved C20 73.6 mm to (68.0, 71.2), turned to 270 degrees
- moved C37 73.5 mm to (68.0, 71.3), turned to 270 degrees
- moved TP21 71.5 mm to (70.0, 25.0)
- moved Q5 69.3 mm to (7.00, 11.0), flipped to the top, turned to 180 degrees
- moved Q6 69.3 mm to (21.0, 11.0), turned to 180 degrees
- moved TP24 64.8 mm to (67.0, 25.0)
- moved Q7 62.8 mm to (35.0, 11.0), flipped to the top, turned to 180 degrees
- moved JP4 51.0 mm to (92.4, 40.2), turned to 0 degrees
- moved R10 47.5 mm to (7.00, 28.0), flipped to the top, turned to 0 degrees
- moved R13 42.4 mm to (20.8, 28.5), turned to 0 degrees
- moved C13 38.7 mm to (48.4, 65.0)
- moved C30 38.3 mm to (69.0, 40.0)
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Connections:
- removed net LATCH_CLK: IC1.11, U4.32
- removed net LATCH_DAT: IC1.14, U4.12
- removed net LATCH_LAT: IC1.12, U4.14
- removed net N$17: IC1.2, Q8.4
- removed net N$19: IC1.3, Q9.2
- removed net N$22: IC1.4, Q9.4
- removed net N$24: IC1.5, Q10.2
- removed net N$26: IC1.6, Q10.4
- removed net N$28: LED1.A, Q11.7, Q11.8
- removed net N$29: LED2.A, Q11.5, Q11.6
- removed net N$30: LED2.C, R29.2
- removed net N$31: LED1.C, R28.2
- new net #CS_EXP: IC2.25, J1.5
- new net ATMEGA_TO_FTDI: IC2.10, JP1.5
- new net EXP_MISO: IC2.2, J1.1
- new net EXP_MOSI: IC2.1, J1.4
- new net EXP_SCK: IC2.3, J1.3
- new net FTDI_TO_ATMEGA: IC2.9, JP1.4
- new net N$10: IC2.43, R8.D1
- new net N$12: IC2.44, R9.A1
- new net N$13: IC2.26, R9.B1
- new net N$14: IC2.36, R9.D1
- new net N$6: IC2.40, R8.A1
- new net N$7: IC2.41, R8.B1
- new net N$8: IC2.42, R8.C1
- new net TCK: IC2.21, JP2.1
- new net TDI: IC2.24, JP2.9
- new net TDO: IC2.23, JP2.3
- new net TMS: IC2.22, JP2.5
- net #CS1: now also IC2.33; no longer U4.26
- net #CS2: now also IC2.34; no longer U4.27
- net #CS3: now also IC2.35; no longer U4.28
- net 3.3V: now also U$15.1; no longer U6.1
- net 5V: now also IC2.17, IC2.27, IC2.38, IC2.5, J1.2, JP2.4; no longer IC1.10, IC1.16, JP2.2, Q10.1, Q10.3, Q11.1, Q11.3, Q8.1, Q8.3, Q9.1, Q9.3, U4.18, U4.4, U4.6
- net ATMEGA_TO_MOTE_3V: now also U$15.3; no longer U6.3
- net ATMEGA_TO_MOTE_5V: now also IC2.12; no longer JP1.5, U4.31
- net GATE1: now also R8.A2; no longer Q8.7, Q8.8
- net GATE2: now also R8.B2; no longer Q8.5, Q8.6
- net GATE3: now also R8.C2; no longer Q9.7, Q9.8
- net GATE4: now also R8.D2; no longer Q9.5, Q9.6
- net GATE5: now also R9.A2; no longer Q10.7, Q10.8
- net GATE6: now also R9.B2; no longer Q10.5, Q10.6
- net GND: now also IC2.18, IC2.28, IC2.39, IC2.6, J1.6, JP2.10, JP2.2, LED1.C, LED2.C, U$15.10, U$15.16; no longer IC1.13, IC1.8, JP2.6, R28.1, R29.1, U4.21, U4.3, U4.5, U6.10, U6.16
- net LED1: now also LED1.A, R9.C2; no longer IC1.15, Q11.2
- net LED2: now also LED2.A, R9.D2; no longer IC1.7, Q11.4
- net MISO: no longer JP2.1, U4.16
- net MOSI: no longer JP2.4, U4.15
- net MOTE_RADIO_INHIBIT_5V: now also IC2.30; no longer U4.23
- net MOTE_RESETN_3V: now also U$15.5; no longer U6.5
- net MOTE_RESETN_5V: now also IC2.20; no longer U4.11
- net MOTE_RX_CTSN_5V: now also IC2.19; no longer U4.10
- net MOTE_RX_RTSN_5V: now also IC2.15; no longer U4.9
- net MOTE_SLEEPN_5V: now also IC2.31; no longer U4.24
- net MOTE_TIMEN_5V: now also IC2.32; no longer U4.25
- net MOTE_TO_ATMEGA_3V: now also U$15.2; no longer U6.2
- net MOTE_TO_ATMEGA_5V: now also IC2.11; no longer JP1.4, U4.30
- net MOTE_TX_CTSN_5V: now also IC2.14; no longer U4.2
- net MOTE_TX_RTSN_5V: now also IC2.13; no longer U4.1
- net N$1: now also IC2.7; no longer U4.7
- net N$16: now also IC2.37, R9.C1; no longer IC1.1, Q8.2
- net N$3: now also IC2.8; no longer U4.8
- net RST: now also IC2.4, JP2.6; no longer JP2.5, U4.29
- net SCLK: no longer JP2.3, U4.17
- net XIN: now also IC2.16; no longer U4.13
Routing:
- net GND: track 618.2 -> 0.00 mm, vias 3 -> 0
- net 5V: track 313.8 -> 0.00 mm, vias 2 -> 0
- net #CS1: track 171.3 -> 0.00 mm, vias 3 -> 0
- net 3.3V: track 117.4 -> 0.00 mm
- net SCLK: track 87.1 -> 0.00 mm, vias 5 -> 0
- net MISO: track 86.0 -> 0.00 mm, vias 3 -> 0
- net GATE2: track 79.3 -> 0.00 mm
- net XIN: track 75.9 -> 0.00 mm, vias 4 -> 0
- net MOTE_RESETN_3V: track 75.3 -> 0.00 mm, vias 2 -> 0
- net V+: track 71.1 -> 0.00 mm, vias 3 -> 0
- net MOTE_RX_CTSN_3V: track 65.5 -> 0.00 mm, vias 5 -> 0
- net MOSI: track 59.9 -> 0.00 mm
- net MOTE_TO_ATMEGA_3V: track 58.7 -> 0.00 mm, vias 3 -> 0
- net RST: track 56.1 -> 0.00 mm, vias 1 -> 0
- net V-: track 55.4 -> 0.00 mm, vias 5 -> 0
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- added copper zone on layer 15, net 5V
- added copper zone on layer 2, net GND

Commit message: Ready to route
Parts:
- removed H1, H2, H3, H4, H5, H6, NEUT1, NEUT2: 1P_HOLE, Cool_Electricity:14GAUGE_HOLE
- removed JP3: (no value), jumper:JP2
- added AC1, AC2, AC3, AC4, AC5, AC6: AC_OUTLET, Cool_Electricity:3-213598-2
- added EARTH, NEUT: 1P_HOLE, Cool_Electricity:14GAUGE_HOLE
- U8, U9: value SN74VC4245A -> SN74LVC4245A
- moved R19 144.0 mm to (177.7, 39.4), flipped to the top
- moved C19 133.6 mm to (175.0, 59.0), turned to 180 degrees
- moved C15 131.1 mm to (174.5, 54.0), turned to 90 degrees
- moved R37 131.0 mm to (175.0, 56.8), turned to 180 degrees
- moved R20 130.2 mm to (170.3, 39.5), flipped to the top
- moved Q6 129.1 mm to (149.0, 28.0), turned to 0 degrees
- moved Q7 128.8 mm to (150.0, 69.0)
- moved R16 127.9 mm to (149.8, 84.5)
- moved U3 124.1 mm to (167.7, 52.7), turned to 180 degrees
- moved R13 123.9 mm to (143.8, 13.5)
- moved C14 121.9 mm to (160.0, 54.0), turned to 270 degrees
- moved R21 120.5 mm to (163.2, 39.5), flipped to the top, turned to 180 degrees
- moved C13 117.2 mm to (163.3, 41.6), flipped to the top, turned to 180 degrees
- moved Q5 114.4 mm to (105.0, 70.0)
- moved R10 113.4 mm to (105.0, 85.0)
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Connections:
- removed net N$18: H2.P$1, Q3.2
- removed net N$20: H3.P$1, Q4.2
- removed net N$21: H4.P$1, Q5.2
- removed net N$23: H5.P$1, Q6.2
- removed net N$25: H6.P$1, Q7.2
- removed net N$5: JP3.2, U8.22, U9.22
- removed net N$9: H1.P$1, Q2.2
- new net EARTH: AC1.3, AC2.3, AC3.3, AC4.3, AC5.3, AC6.3, EARTH.P$1
- new net HOT1: AC1.2, Q2.2
- new net HOT2: AC2.2, Q3.2
- new net HOT3: AC3.2, Q4.2
- new net HOT4: AC4.2, Q5.2
- new net HOT5: AC5.2, Q6.2
- new net HOT6: AC6.2, Q7.2
- net 5V: now also U8.22; no longer JP3.3
- net GND: now also U9.22; no longer JP3.1
- net NEUTRAL: now also AC1.1, AC2.1, AC3.1, AC4.1, AC5.1, AC6.1, NEUT.P$1; no longer NEUT1.P$1, NEUT2.P$1
Routing:
- net NEUTRAL: track 0.00 -> 522.8 mm
- net EARTH: track 0.00 -> 470.2 mm
- net GND: track 0.00 -> 445.5 mm
- net HOT1: track 0.00 -> 39.5 mm
- net HOT5: track 0.00 -> 37.5 mm
- net HOT3: track 0.00 -> 37.3 mm
- net HOT2: track 0.00 -> 13.8 mm
- net HOT6: track 0.00 -> 13.8 mm
- net HOT4: track 0.00 -> 12.8 mm
- net V+: track 0.00 -> 6.85 mm
- net HRET2: track 0.00 -> 5.79 mm
- net HRET6: track 0.00 -> 5.29 mm
- net HRET4: track 0.00 -> 5.03 mm
- net N$2: track 0.00 -> 4.67 mm
- net HRET5: track 0.00 -> 4.37 mm
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- removed copper zone on layer 15, net 5V
- removed copper zone on layer 2, net GND
Other:
- board size 100 x 80 mm -> 185 x 95 mm
- board text added: "SOLDER 14AWG WIRE ON BUS"
