File: power_strip_monitor/power_strip_monitor_V2.sch (EAGLE design)
At the start: 108 parts, among them Q1 4.096MHz, U1 CS5467, U10 LTP5901, U2 CS5467, U3 CS5467, U4 ATMEGA168, U5 LNK302, U6 XBEE-1B1, U8 SN74VC4245A, U9 SN74VC4245A

Commit message: Finished, now optimize
Parts:
- removed C32: 22p, SparkFun:CAP0603
- removed NEUTRAL: 1P_HOLE, Cool_Electricity:1P_HOLE
- added C30: 22p, SparkFun:CAP0603
- added HOT: 1P_HOLE, Cool_Electricity:1P_HOLE
- added IC1: 74HC595D, 74xx-eu:74HC595D
- added Q10, Q11, Q8, Q9: (no value), Cool_Electricity:DUAL-MOSFET-PCHANNELSOT563
- added Q2, Q3, Q4, Q5, Q6, Q7: BTA312B-800E, Cool_Electricity:TRIACD2PACK
- added R28, R29: 150, SparkFun:RESISTOR0603
- LED1, LED2: device led:LEDCHIPLED_0805 -> led:LEDCHIP-LED0805
- Q1: value 4.096MHz -> 16.384MHz
- R26: value 10k -> 2k 1%
- R27: value 10k -> 4.06k 1%
- renumbered LINE to NEUT2, LINE1 to NEUT1, N1 to H1, N2 to H2, N3 to H3, N4 to H4, N5 to H5, N6 to H6
Connections:
- net HOT renamed NEUTRAL
- removed net NRET1: H1.1, R1.2, R2.2
- removed net NRET2: H2.1, R4.2, R5.2
- removed net NRET3: H3.1, R7.2, R8.2
- removed net NRET4: H4.1, R10.2, R11.2
- removed net NRET5: H5.1, R13.2, R14.2
- removed net NRET6: H6.1, R16.2, R17.2
- new net GATE1: Q2.G, Q8G1.S
- new net GATE2: Q3.G, Q8G2.S
- new net GATE3: Q4.G, Q9G1.S
- new net GATE4: Q5.G, Q9G2.S
- new net GATE5: Q10G1.S, Q6.G
- new net GATE6: Q10G2.S, Q7.G
- new net HRET1: Q2.M1, R1.2, R2.2
- new net HRET2: Q3.M1, R4.2, R5.2
- new net HRET3: Q4.M1, R7.2, R8.2
- new net HRET4: Q5.M1, R10.2, R11.2
- new net HRET5: Q6.M1, R13.2, R14.2
- new net HRET6: Q7.M1, R16.2, R17.2
- new net LATCH_CLK: IC1A.SCK, U4.PD2(INT0)
- new net LATCH_DAT: IC1A.SER, U4.PB0(ICP)
- new net LATCH_LAT: IC1A.RCK, U4.PB2(SS/OC1B)
- new net LED1: IC1A.QA, Q11G2.G
- new net LED2: IC1A.QH, Q11G1.G
- new net N$18: H2.1, Q3.M2
- new net N$19: IC1A.QD, Q9G1.G
- new net N$20: H3.1, Q4.M2
- new net N$21: H4.1, Q5.M2
- new net N$22: IC1A.QE, Q9G2.G
- new net N$23: H5.1, Q6.M2
- new net N$24: IC1A.QF, Q10G1.G
- new net N$25: H6.1, Q7.M2
- new net N$26: IC1A.QG, Q10G2.G
- new net N$28: LED1.A, Q11G2.S
- new net N$29: LED2.A, Q11G1.S
- new net N$30: LED2.C, R29.2
- new net N$31: LED1.C, R28.2
- new net N$9: H1.1, Q2.M2
- net 5V: now also IC1A.SCL, IC1P.VCC, Q10G1.D, Q10G2.D, Q11G1.D, Q11G2.D, Q8G1.D, Q8G2.D, Q9G1.D, Q9G2.D
- net GND: now also C30.2, HOT.1, IC1A.G, IC1P.GND, R28.1, R29.1; no longer C32.2, LED1.C, LED2.C, NEUTRAL.1
- net N$1: now also C30.1, Q1.2, U4.PB6(XTAL1/TOSC1); no longer LED2.A, U4.PB1(OC1A)
- net N$16: now also IC1A.QB, Q8G1.G; no longer C31.1, Q1.2, U4.PB6(XTAL1/TOSC1)
- net N$17: now also IC1A.QC, Q8G2.G; no longer C32.1, Q1.1, U4.PB7(XTAL2/TOSC2)
- net N$3: now also C31.1, Q1.1, U4.PB7(XTAL2/TOSC2); no longer LED1.A, U4.PB2(SS/OC1B)
- net XIN: now also U4.PB1(OC1A); no longer U4.PB0(ICP)
Other:
- note added: "NOTE: GND=HOT"
- note removed: "NOTE: GND=NEUTRAL"
- moved on the sheet: C31, LED1, LED2, Q1

Commit message: components placed
Parts:
- removed C10, C11, C12, C4, C5, C6, C7, C8, C9: 10n, SparkFun:CAP0603
- removed C16, C17: 4.7uF 400V, SparkFun-Passives:CAP_POLPTH3
- removed C18: 100n, SparkFun:CAP0603
- removed C22: 10u 35V, SparkFun-Capacitors:CAP1206
- removed D1: S1M-13-F, Cool_Electricity:DIODESMA-KIT
- removed D2, D3: ES1D, Cool_Electricity:DIODESMA-KIT
- removed L1: ELL-6UH102M, Cool_Electricity:INDUCTORELL6RH
- removed L2: PM5022-102M-RC, Cool_Electricity:INDUCTORPM5022
- removed R11, R12, R14, R15, R17, R18, R8, R9: 330 1%, SparkFun:RESISTOR0603
- removed R22, R23, R24, R46: 10k, SparkFun:RESISTOR0603
- removed R26: 2k 1%, SparkFun:RESISTOR0603
- removed R27: 4.06k 1%, SparkFun:RESISTOR0603
- removed TP1, TP10, TP11, TP12, TP18, TP2, TP3, TP4, TP5, TP6, TP7, TP8, TP9: TESTPOINTSMALLEST, WSNlib:TESTPOINTSMALLEST
- C1, C2, C3: value 10n -> CAP_ARRAY; device SparkFun:CAP0603 -> Cool_Electricity:CAP_ARRAY
- R2, R3, R5: value 330 1% -> 220 1%; device SparkFun:RESISTOR0603 -> Cool_Electricity:RESISTOR-ARRAY
- R25: value FKN200JR-73-8R2 -> S14K680; device SparkFun-Resistors:RESISTORPTH-1W -> varistor:S14K680
- R6: value 330 1% -> (none); device SparkFun:RESISTOR0603 -> Cool_Electricity:RESISTOR-ARRAY
- U5: value LNK302 -> RAC01_02-SC; device Cool_Electricity:LNK302 -> Cool_Electricity:RAC01_02-SC
Connections:
- removed net N$10: C22.1, D3.C, R27.1
- removed net N$12: C18.2, U5.BP
- removed net N$13: C18.1, C22.2, D2.C, L2.1, R26.1, U5.S@1, U5.S@2, U5.S@3, U5.S@4
- removed net N$14: R26.2, R27.2, U5.FB
- removed net N$6: D1.A, R25.2
- removed net N$7: C16.+, D1.C, L1.1
- removed net N$8: C17.+, L1.2, U5.D
- net #CS1: now also R6A.1; no longer R24.1
- net #CS2: now also R6B.1; no longer R23.1
- net #CS3: now also R6C.1; no longer R22.1
- net 5V: now also R6A.2, R6B.2, R6C.2, R6D.2, U5.VOUT+; no longer D3.A, L2.2, R22.2, R23.2, R24.2, R46.2
- net GND: now also C1A.2, C1B.2, C1C.2, C1D.2, C2A.2, C2B.2, C2C.2, C2D.2, C3A.2, C3B.2, C3C.2, C3D.2, R25.1, R2B.1, R2D.1, R3B.1, R3D.1, R5B.1, R5D.1, U5.AC_NEUT, U5.VOUT-; no longer C1.2, C10.1, C11.2, C12.1, C16.-, C17.-, C2.1, C3.2, C4.1, C5.2, C6.1, C7.2, C8.1, C9.2, D2.A, R12.2, R15.2, R18.2, R3.2, R6.2, R9.2
- net HRET1: now also R2A.1; no longer R2.2
- net HRET2: now also R2C.1; no longer R5.2
- net HRET3: now also R3A.1; no longer R8.2
- net HRET4: now also R3C.1; no longer R11.2
- net HRET5: now also R5A.1; no longer R14.2
- net HRET6: now also R5C.1; no longer R17.2
- net I1+: now also C1A.1, R2A.2; no longer C1.1, R2.1, TP2.P$1
- net I1-: now also C1B.1, R2B.2; no longer C2.2, R3.1, TP1.P$1
- net I2+: now also C1C.1, R2C.2; no longer C3.1, R5.1, TP3.P$1
- net I2-: now also C1D.1, R2D.2; no longer C4.2, R6.1, TP4.P$1
- net I3+: now also C2A.1, R3A.2; no longer C5.1, R8.1, TP5.P$1
- net I3-: now also C2B.1, R3B.2; no longer C6.2, R9.1, TP6.P$1
- net I4+: now also C2C.1, R3C.2; no longer C7.1, R11.1, TP7.P$1
- net I4-: now also C2D.1, R3D.2; no longer C8.2, R12.1, TP8.P$1
- net I5+: now also C3A.1, R5A.2; no longer C9.1, R14.1, TP9.P$1
- net I5-: now also C3B.1, R5B.2; no longer C10.2, R15.1, TP10.P$1
- net I6+: now also C3C.1, R5C.2; no longer C11.1, R17.1, TP11.P$1
- net I6-: now also C3D.1, R5D.2; no longer C12.2, R18.1, TP12.P$1
- net NEUTRAL: now also R25.2, U5.AC_LINE; no longer R25.1
- net RST: now also R6D.1; no longer R46.1
- net V+: no longer TP18.P$1

Commit message: Trying to route now
Parts:
- Q10, Q11, Q8, Q9: device Cool_Electricity:DUAL-MOSFET-PCHANNELSOT563 -> Cool_Electricity:DUAL-MOSFET-PCHANNEL2D
Connections:
- net 5V: now also Q10A.S, Q10B.S, Q11A.S, Q11B.S, Q8A.S, Q8B.S, Q9A.S, Q9B.S; no longer Q10G1.D, Q10G2.D, Q11G1.D, Q11G2.D, Q8G1.D, Q8G2.D, Q9G1.D, Q9G2.D
- net GATE1: now also Q8A.D@1, Q8A.D@2; no longer Q8G1.S
- net GATE2: now also Q8B.D@1, Q8B.D@2; no longer Q8G2.S
- net GATE3: now also Q9A.D@1, Q9A.D@2; no longer Q9G1.S
- net GATE4: now also Q9B.D@1, Q9B.D@2; no longer Q9G2.S
- net GATE5: now also Q10A.D@1, Q10A.D@2; no longer Q10G1.S
- net GATE6: now also Q10B.D@1, Q10B.D@2; no longer Q10G2.S
- net LED1: now also Q11A.G; no longer Q11G2.G
- net LED2: now also Q11B.G; no longer Q11G1.G
- net N$16: now also Q8A.G; no longer Q8G1.G
- net N$17: now also Q8B.G; no longer Q8G2.G
- net N$19: now also Q9A.G; no longer Q9G1.G
- net N$22: now also Q9B.G; no longer Q9G2.G
- net N$24: now also Q10A.G; no longer Q10G1.G
- net N$26: now also Q10B.G; no longer Q10G2.G
- net N$28: now also Q11A.D@1, Q11A.D@2; no longer Q11G2.S
- net N$29: now also Q11B.D@1, Q11B.D@2; no longer Q11G1.S

Commit message: Latest Powerstrip changes
Parts:
- removed IC1: 74HC595D, 74xx-eu:74HC595D
- removed Q10, Q11, Q8, Q9: (no value), Cool_Electricity:DUAL-MOSFET-PCHANNEL2D
- removed R28, R29: 150, SparkFun:RESISTOR0603
- removed U4: ATMEGA168, SparkFun:ATMEGA168
- removed U6: XBEE-1B1, SparkFun:XBEE-1B1
- added IC2: ATMEGA644A, atmel:ATMEGA644A
- added J1: EXP, SparkFun-Connectors:AVR_SPI_PRG_6PTH
- added R8, R9: 100, Cool_Electricity:RESISTOR-ARRAY
- added U$15: XBEE-1B3, SparkFun-RF:XBEE-1B3
- JP2: value AVR_SPI_PRG_6NS -> JTAG; device SparkFun:AVR_SPI_PRG_6NS -> SparkFun-Connectors:M05X2PTH
- LED1, LED2: device led:LEDCHIP-LED0805 -> led:LEDCHIPLED_0805
Connections:
- removed net LATCH_CLK: IC1A.SCK, U4.PD2(INT0)
- removed net LATCH_DAT: IC1A.SER, U4.PB0(ICP)
- removed net LATCH_LAT: IC1A.RCK, U4.PB2(SS/OC1B)
- removed net N$17: IC1A.QC, Q8B.G
- removed net N$19: IC1A.QD, Q9A.G
- removed net N$22: IC1A.QE, Q9B.G
- removed net N$24: IC1A.QF, Q10A.G
- removed net N$26: IC1A.QG, Q10B.G
- removed net N$28: LED1.A, Q11A.D@1, Q11A.D@2
- removed net N$29: LED2.A, Q11B.D@1, Q11B.D@2
- removed net N$30: LED2.C, R29.2
- removed net N$31: LED1.C, R28.2
- new net #CS_EXP: IC2.(PCINT22/TOSC1)PC6, J1.5
- new net ATMEGA_TO_FTDI: IC2.(PCINT25/TXD0)PD1, JP1.RXD
- new net EXP_MISO: IC2.(PCINT14/MISO)PB6, J1.1
- new net EXP_MOSI: IC2.(PCINT13/MOSI)PB5, J1.4
- new net EXP_SCK: IC2.(PCINT15/SCK)PB7, J1.3
- new net FTDI_TO_ATMEGA: IC2.(PCINT24/RXD0)PD0, JP1.TXD
- new net N$10: IC2.(PCINT11/OC0A/AIN1)PB3, R8D.1
- new net N$12: IC2.(PCINT12/OC0B/!SS!)PB4, R9A.1
- new net N$13: IC2.(PCINT23/TOSC2)PC7, R9B.1
- new net N$14: IC2.(PCINT1/ADC1)PA1, R9D.1
- new net N$6: IC2.(PCINT8/XCK0/T0)PB0, R8A.1
- new net N$7: IC2.(PCINT9/CLKO/T1)PB1, R8B.1
- new net N$8: IC2.(PCINT10/INT2/AIN0)PB2, R8C.1
- new net TCK: IC2.(PCINT18/TCK)PC2, JP2.1
- new net TDI: IC2.(PCINT21/TDI)PC5, JP2.9
- new net TDO: IC2.(PCINT20/TDO)PC4, JP2.3
- new net TMS: IC2.(PCINT19/TMS)PC3, JP2.5
- net #CS1: now also IC2.(PCINT4/ADC4)PA4; no longer U4.PC3(ADC3)
- net #CS2: now also IC2.(PCINT3/ADC3)PA3; no longer U4.PC4(ADC4/SDA)
- net #CS3: now also IC2.(PCINT2/ADC2)PA2; no longer U4.PC5(ADC5/SCL)
- net 3.3V: now also U$15.VDD; no longer U6.VDD
- net 5V: now also IC2.AVCC, IC2.VCC, IC2.VCC@1, IC2.VCC@2, J1.2, JP2.4; no longer IC1A.SCL, IC1P.VCC, JP2.2, Q10A.S, Q10B.S, Q11A.S, Q11B.S, Q8A.S, Q8B.S, Q9A.S, Q9B.S, U4.AVCC, U4.VCC@1, U4.VCC@2
- net ATMEGA_TO_MOTE_3V: now also U$15.DIN; no longer U6.DIN
- net ATMEGA_TO_MOTE_5V: now also IC2.(PCINT27/INT1)PD3; no longer JP1.RXD, U4.PD1(TXD)
- net GATE1: now also R8A.2; no longer Q8A.D@1, Q8A.D@2
- net GATE2: now also R8B.2; no longer Q8B.D@1, Q8B.D@2
- net GATE3: now also R8C.2; no longer Q9A.D@1, Q9A.D@2
- net GATE4: now also R8D.2; no longer Q9B.D@1, Q9B.D@2
- net GATE5: now also R9A.2; no longer Q10A.D@1, Q10A.D@2
- net GATE6: now also R9B.2; no longer Q10B.D@1, Q10B.D@2
- net GND: now also IC2.GND, IC2.GND@1, IC2.GND@2, IC2.GND@3, J1.6, JP2.10, JP2.2, LED1.C, LED2.C, U$15.GND, U$15.RTS; no longer IC1A.G, IC1P.GND, JP2.6, R28.1, R29.1, U4.AGND, U4.GND@1, U4.GND@2, U6.GND, U6.RTS
- net LED1: now also LED1.A, R9C.2; no longer IC1A.QA, Q11A.G
- net LED2: now also LED2.A, R9D.2; no longer IC1A.QH, Q11B.G
- net MISO: no longer JP2.1, U4.PB4(MISO)
- net MOSI: no longer JP2.4, U4.PB3(MOSI/OC2)
- net MOTE_RADIO_INHIBIT_5V: now also IC2.(PCINT7/ADC7)PA7; no longer U4.PC0(ADC0)
- net MOTE_RESETN_3V: now also U$15.RESET; no longer U6.RESET
- net MOTE_RESETN_5V: now also IC2.(PCINT17/SDA)PC1; no longer U4.PD7(AIN1)
- net MOTE_RX_CTSN_5V: now also IC2.(PCINT16/SCL)PC0; no longer U4.PD6(AIN0)
- net MOTE_RX_RTSN_5V: now also IC2.(PCINT30/OC2B/ICP)PD6; no longer U4.PD5(T1)
- net MOTE_SLEEPN_5V: now also IC2.(PCINT6/ADC6)PA6; no longer U4.PC1(ADC1)
- net MOTE_TIMEN_5V: now also IC2.(PCINT5/ADC5)PA5; no longer U4.PC2(ADC2)
- net MOTE_TO_ATMEGA_3V: now also U$15.DOUT; no longer U6.DOUT
- net MOTE_TO_ATMEGA_5V: now also IC2.(PCINT26/INT0)PD2; no longer JP1.TXD, U4.PD0(RXD)
- net MOTE_TX_CTSN_5V: now also IC2.(PCINT29/OC1A)PD5; no longer U4.PD4(XCK/T0)
- net MOTE_TX_RTSN_5V: now also IC2.(PCINT28/OC1B)PD4; no longer U4.PD3(INT1)
- net N$1: now also IC2.XTAL2; no longer U4.PB6(XTAL1/TOSC1)
- net N$16: now also IC2.(PCINT0/ADC0)PA0, R9C.1; no longer IC1A.QB, Q8A.G
- net N$3: now also IC2.XTAL1; no longer U4.PB7(XTAL2/TOSC2)
- net RST: now also IC2.RESET, JP2.6; no longer JP2.5, U4.PC6(/RESET)
- net SCLK: no longer JP2.3, U4.PB5(SCK)
- net XIN: now also IC2.(PCINT31/OC2A)PD7; no longer U4.PB1(OC1A)
Other:
- note removed: "AN0"
- note removed: "AN1"
- note removed: "AN2"
- note removed: "AN3"
- note removed: "AN4"
- note removed: "AN5"
- note removed: "DIG0"
- note removed: "DIG1"
- note removed: "DIG10 (PWM)"
- note removed: "DIG11 (PWM)"
- note removed: "DIG12"
- note removed: "DIG13"
- note removed: "DIG14"
- note removed: "DIG15"
- note removed: "DIG16"
- note removed: "DIG17"
- note removed: "DIG18"
- note removed: "DIG19"
- note removed: "DIG2"
- note removed: "DIG3"
- note removed: "DIG4"
- note removed: "DIG5 (PWM)"
- note removed: "DIG6 (PWM)"
- note removed: "DIG7"
- note removed: "DIG8"
- note removed: "DIG9 (PWM)"
- moved on the sheet: C30, C31, C33, C34, C41, LED1, LED2, Q1, R6D

Commit message: Ready to route
Parts:
- removed H1, H2, H3, H4, H5, H6, NEUT1, NEUT2: 1P_HOLE, Cool_Electricity:1P_HOLE
- removed JP3: (no value), jumper:JP2E
- added AC1, AC2, AC3, AC4, AC5, AC6: AC_OUTLET, Cool_Electricity:AC_OUTLET
- added EARTH, NEUT: 1P_HOLE, Cool_Electricity:1P_HOLE
- U8, U9: value SN74VC4245A -> SN74LVC4245A
Connections:
- removed net N$18: H2.1, Q3.M2
- removed net N$20: H3.1, Q4.M2
- removed net N$21: H4.1, Q5.M2
- removed net N$23: H5.1, Q6.M2
- removed net N$25: H6.1, Q7.M2
- removed net N$5: JP3.2, U8.#OE, U9.#OE
- removed net N$9: H1.1, Q2.M2
- new net EARTH: AC1.EARTH, AC2.EARTH, AC3.EARTH, AC4.EARTH, AC5.EARTH, AC6.EARTH, EARTH.1
- new net HOT1: AC1.L, Q2.M2
- new net HOT2: AC2.L, Q3.M2
- new net HOT3: AC3.L, Q4.M2
- new net HOT4: AC4.L, Q5.M2
- new net HOT5: AC5.L, Q6.M2
- new net HOT6: AC6.L, Q7.M2
- net 5V: now also U8.#OE; no longer JP3.3
- net GND: now also U9.#OE; no longer JP3.1
- net NEUTRAL: now also AC1.N, AC2.N, AC3.N, AC4.N, AC5.N, AC6.N, NEUT.1; no longer NEUT1.1, NEUT2.1

Commit message: ready for mfg? BOM needs fixing
Parts:
- C1, C2, C3: value CAP_ARRAY -> 10n
- R6: value (none) -> 10k
- U7: value (none) -> LT1761ES5-3.3
- renumbered J1 to EXP, JP1 to FTDI, JP2 to JTAG, U$15 to U15
