File: dust_environment_sensor/dust_environment_sensor_v2.sch (EAGLE design)
At the start: 45 parts, among them IC2 ATMEGA644A, J1 3.6V Lithium C cell, J2 EXP, J3 XBEE_1-10SMT, J4 XBEE_11-20SMT, U1 LTP5901, U2 LIS3DH, U3 SI7005, U4 TSL2560, U5 AMN41121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

Commit message: changes for v2
Parts:
- removed JP1: 87758-1016, con-molex:87758-1016
- removed U1: LTP5901, Cool_Electricity:LTP5901
- added C16, C17: 1u, rcl:C-EUC0603
- added C18: 100n, rcl:C-EUC0603
- added R3: 15, resistor:R-US_R0603
- added U7: MCP1700-3.3V, Cool_Electricity:MCP1700
- C6: value 100n -> 680u; device rcl:C-EUC0603 -> SparkFun-Capacitors:CAP_POL7343
- R5: value 0R -> 0R DNP
Connections:
- removed net FLASH_P_ENN: JP1-2.S, U1.FLASH_P_ENN
- removed net IPCS_MISO: JP1-5.S, U1.IPCS_MISO/GPIO6
- removed net IPCS_MOSI: JP1-4.S, U1.IPCS_MOSI/GPIO5
- removed net IPCS_SCK: JP1-3.S, U1.IPCS_SCK/GPIO4
- removed net IPCS_SSN: JP1-1.S, U1.IPCS_SSN/GPIO3
- removed net MOTE_CLI_RX: JP1-10.S, U1.UARTC0_RX
- removed net MOTE_CLI_TX: JP1-9.S, U1.UARTC0_TX
- removed net MOTE_RADIO_INHIBIT: IC2.(PCINT5/ADC5)PA5, U1.RADIO_INHIBIT
- removed net MOTE_RX_CTSN: IC2.(PCINT8/XCK0/T0)PB0, U1.UART_RX_CTSN
- removed net MOTE_TIMEN: IC2.(PCINT3/ADC3)PA3, U1.TIMEN
- removed net MOTE_TX_RTSN: IC2.(PCINT10/INT2/AIN0)PB2, U1.UART_TX_RTSN
- new net HUMID_VCC: IC2.(PCINT3/ADC3)PA3, R3.1
- new net MOTE_ASSOC: IC2.(PCINT9/CLKO/T1)PB1, J4.ASSOC/AD5/DIO5
- new net MOTE_STATUS: IC2.(PCINT10/INT2/AIN0)PB2, J4.ON/!SLEEP
- new net N$11: C5.1, R3.2, U3.VDD
- net GND: now also C16.2, C17.2, C18.1, C6.-, U7.GND; no longer C6.2, JP1-8.S, U1.GND@1, U1.GND@2, U1.GND@3, U1.GND@4, U1.GND@5, U1.GND@6, U1.GND@7, U1.GND@8, U1.GND@9
- net MOTE_API_RX: no longer U1.UART_RX
- net MOTE_API_TX: no longer U1.UART_TX
- net MOTE_RESETN: now also IC2.(PCINT4/ADC4)PA4; no longer JP1-6.S, U1.RESETN
- net MOTE_RX_RTSN: no longer U1.UART_RX_RTSN
- net MOTE_SLEEPN: now also IC2.(PCINT5/ADC5)PA5; no longer IC2.(PCINT4/ADC4)PA4, U1.SLEEPN
- net MOTE_TX_CTSN: now also IC2.(PCINT8/XCK0/T0)PB0, J4.!CTS!/DIO7; no longer IC2.(PCINT9/CLKO/T1)PB1, U1.UART_TX_CTSN
- net VBATT: now also C16.1, J2.2, JP8.VCC, U7.VIN
- net VCC: now also C17.1, C18.2, C6.+, U7.VOUT; no longer C5.1, C6.1, J2.2, JP1-7.S, U1.VSUPPLY, U3.VDD

Commit message: Test golden version of ES2
Parts:
- added U1: TSL2560T, Cool_Electricity:TSL2560T
- C3: device rcl:C-USC0603 -> rcl:C-EUC0603
- U4: value TSL2560 -> TSL2560CL; device Cool_Electricity:TSL2560 -> Cool_Electricity:TSL2560CL
Connections:
- net GND: now also U1.ADDR, U1.GND
- net I2C_SCL: now also U1.SCL
- net I2C_SDA: now also U1.SDA
- net LIGHT_INT: now also U1.INT
- net VCC: now also U1.VDD
Changed lines of the file:
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@@
 <part name="U2" library="Cool_Electricity" deviceset="LIS3DH" device=""/>
 <part name="U3" library="Cool_Electricity" deviceset="SI7005" device=""/>
-<part name="U4" library="Cool_Electricity" deviceset="TSL2560" device=""/>
+<part name="U4" library="Cool_Electricity" deviceset="TSL2560" device="CL"/>
 <part name="GND1" library="supply1" deviceset="GND" device=""/>
 <part name="GND2" library="supply1" deviceset="GND" device=""/>
@@
 <part name="P+5" library="supply1" deviceset="VCC" device=""/>
 <part name="C2" library="rcl" deviceset="C-US" device="C0603" value="10u"/>
-<part name="C3" library="rcl" deviceset="C-US" device="C0603" value="100n"/>
 <part name="C4" library="SparkFun-Capacitors" deviceset="CAP_POL" device="1206-KIT" value="100u"/>
 <part name="GND8" library="supply1" deviceset="GND" device=""/>
@@
 <part name="C18" library="rcl" deviceset="C-EU" device="C0603" value="100n"/>
 <part name="GND4" library="supply1" deviceset="GND" device=""/>
+<part name="U1" library="Cool_Electricity" deviceset="TSL2560" device="T"/>
+<part name="GND5" library="supply1" deviceset="GND" device=""/>
+<part name="P+1" library="supply1" deviceset="VCC" device=""/>
+<part name="C3" library="rcl" deviceset="C-EU" device="C0603" value="100n"/>
 </parts>
 <sheets>
@@
 <instance part="P+5" gate="VCC" x="215.9" y="116.84"/>
 <instance part="C2" gate="G$1" x="220.98" y="109.22"/>
-<instance part="C3" gate="G$1" x="307.34" y="88.9"/>
 <instance part="C4" gate="G$1" x="342.9" y="7.62"/>
 <instance part="GND8" gate="1" x="142.24" y="35.56"/>
@@
 <instance part="C18" gate="G$1" x="45.72" y="210.82" rot="R90"/>
 <instance part="GND4" gate="1" x="40.64" y="210.82" rot="R270"/>
+<instance part="U1" gate="G$1" x="279.4" y="104.14"/>
+<instance part="GND5" gate="1" x="297.18" y="99.06"/>
+<instance part="P+1" gate="VCC" x="297.18" y="111.76"/>
+<instance part="C3" gate="G$1" x="307.34" y="88.9"/>
 </instances>
 <busses>
@@
 <wire x1="292.1" y1="81.28" x2="294.64" y2="81.28" width="0.1524" layer="91"/>
 <wire x1="294.64" y1="81.28" x2="294.64" y2="76.2" width="0.1524" layer="91"/>
-<pinref part="C3" gate="G$1" pin="2"/>
 <wire x1="307.34" y1="83.82" x2="307.34" y2="76.2" width="0.1524" layer="91"/>
 <wire x1="307.34" y1="76.2" x2="294.64" y2="76.2" width="0.1524" layer="91"/>
@@
 <wire x1="294.64" y1="83.82" x2="294.64" y2="81.28" width="0.1524" layer="91"/>
 <junction x="294.64" y="81.28"/>
+<pinref part="C3" gate="G$1" pin="2"/>
 </segment>
 <segment>
@@
 <pinref part="GND4" gate="1" pin="GND"/>
 </segment>
+<segment>
+<pinref part="U1" gate="G$1" pin="GND"/>
+<pinref part="GND5" gate="1" pin="GND"/>
+<wire x1="297.18" y1="101.6" x2="294.64" y2="101.6" width="0.1524" layer="91"/>
+<pinref part="U1" gate="G$1" pin="ADDR"/>
+<wire x1="294.64" y1="101.6" x2="292.1" y2="101.6" width="0.1524" layer="91"/>
+<wire x1="292.1" y1="104.14" x2="294.64" y2="104.14" width="0.1524" layer="91"/>
+<wire x1="294.64" y1="104.14" x2="294.64" y2="101.6" width="0.1524" layer="91"/>
+<junction x="294.64" y="101.6"/>
+</segment>
 </net>
 <net name="VCC" class="0">
@@
 </segment>
 <segment>
-<pinref part="C3" gate="G$1" pin="1"/>
 <pinref part="P+2" gate="VCC" pin="VCC"/>
 <wire x1="307.34" y1="91.44" x2="302.26" y2="91.44" width="0.1524" layer="91"/>
@@
 <wire x1="292.1" y1="91.44" x2="292.1" y2="86.36" width="0.1524" layer="91"/>
 <junction x="302.26" y="91.44"/>
+<pinref part="C3" gate="G$1" pin="1"/>
 </segment>
 <segment>
@@
 <junction x="50.8" y="203.2"/>
 </segment>
+<segment>
+<pinref part="U1" gate="G$1" pin="VDD"/>
+<pinref part="P+1" gate="VCC" pin="VCC"/>
+<wire x1="292.1" y1="106.68" x2="297.18" y2="106.68" width="0.1524" layer="91"/>
+<wire x1="297.18" y1="106.68" x2="297.18" y2="109.22" width="0.1524" layer="91"/>
+</segment>
 </net>
 <net name="N$1" class="0">
@@
 <segment>
 <pinref part="U4" gate="G$1" pin="SCL"/>
-<wire x1="264.16" y1="86.36" x2="236.22" y2="86.36" width="0.1524" layer="91"/>
+<wire x1="264.16" y1="86.36" x2="256.54" y2="86.36" width="0.1524" layer="91"/>
 <label x="236.22" y="86.36" size="1.778" layer="95"/>
+<pinref part="U1" gate="G$1" pin="SCL"/>
+<wire x1="256.54" y1="86.36" x2="236.22" y2="86.36" width="0.1524" layer="91"/>
+<wire x1="264.16" y1="106.68" x2="256.54" y2="106.68" width="0.1524" layer="91"/>
+<wire x1="256.54" y1="106.68" x2="256.54" y2="86.36" width="0.1524" layer="91"/>
+<junction x="256.54" y="86.36"/>
 </segment>
 <segment>
@@
 <segment>
 <pinref part="U4" gate="G$1" pin="SDA"/>
-<wire x1="264.16" y1="83.82" x2="236.22" y2="83.82" width="0.1524" layer="91"/>
+<wire x1="264.16" y1="83.82" x2="259.08" y2="83.82" width="0.1524" layer="91"/>
 <label x="236.22" y="83.82" size="1.778" layer="95"/>
+<pinref part="U1" gate="G$1" pin="SDA"/>
+<wire x1="259.08" y1="83.82" x2="236.22" y2="83.82" width="0.1524" layer="91"/>
+<wire x1="264.16" y1="104.14" x2="259.08" y2="104.14" width="0.1524" layer="91"/>
+<wire x1="259.08" y1="104.14" x2="259.08" y2="83.82" width="0.1524" layer="91"/>
+<junction x="259.08" y="83.82"/>
 </segment>
 <segment>
@@
 <segment>
 <pinref part="U4" gate="G$1" pin="INT"/>
-<wire x1="264.16" y1="81.28" x2="236.22" y2="81.28" width="0.1524" layer="91"/>
+<wire x1="264.16" y1="81.28" x2="261.62" y2="81.28" width="0.1524" layer="91"/>
 <label x="236.22" y="81.28" size="1.778" layer="95"/>
-</segment>
-<segment>
+<pinref part="U1" gate="G$1" pin="INT"/>
+<wire x1="261.62" y1="81.28" x2="236.22" y2="81.28" width="0.1524" layer="91"/>
+<wire x1="264.16" y1="101.6" x2="261.62" y2="101.6" width="0.1524" layer="91"/>
+<wire x1="261.62" y1="101.6" x2="261.62" y2="81.28" width="0.1524" layer="91"/>
+<junction x="261.62" y="81.28"/>
+</segment>
+<segment>
