File: dust_environment_sensor/dust_environment_sensor_v3.brd (EAGLE design)
At the start: 70 x 70 mm, 49 parts, among them IC2 ATMEGA644A, J1 3.6V Lithium C cell, J2 EXP, J3 XBEE_1-10SMT, J4 XBEE_11-20SMT, U1 TSL2560T, U2 LIS3DH, U3 SI7005, U4 TSL2560CL, U5 AMN41121, U6 L3GD20, U7 MCP1700-3.3V, X2 32.768KHz

Commit message: tiny DES3
Parts:
- removed C13, C15, C5: 100n, rcl:C0603
- removed C14: 10u, rcl:C0603
- removed C7: 4.7u, rcl:C0603
- removed J2: EXP, SparkFun-Connectors:2X3
- removed JP4, JP5, JP6, JP7: M01PTH, SparkFun-Connectors:1X01
- removed R3: 15, resistor:R0603
- removed U3: SI7005, Cool_Electricity:QFN24_SILICON_LABS
- removed U6: L3GD20, Cool_Electricity:LGA16_4X4_ST
- added EXP: M05X2SHD, SparkFun-Connectors:2X5-SHROUDED
- C4: value 100u -> 100n; device SparkFun-Capacitors:EIA3216-KIT -> rcl:C0603
- JP9: device SparkFun-Connectors:AVR_ICSP -> SparkFun-Connectors:2X5-SHROUDED
- U4: value TSL2560CL -> HTU21D; device Cool_Electricity:CL6_TAOS -> Cool_Electricity:HTU21D
- moved R5 55.5 mm to (61.0, 22.0), turned to 0 degrees
- moved STANDOFF1 53.4 mm to (24.0, 65.5)
- moved U5 53.0 mm to (54.4, 19.0), turned to 180 degrees
- moved C16 52.7 mm to (61.0, 16.1), turned to 180 degrees
- moved C12 52.6 mm to (8.50, 17.0), turned to 270 degrees
- moved X2 51.4 mm to (8.50, 20.8), turned to 90 degrees
- moved C11 50.7 mm to (8.50, 24.5), turned to 90 degrees
- moved STANDOFF3 50.1 mm to (42.5, 61.0)
- moved R6 49.4 mm to (60.0, 24.7), turned to 270 degrees
- moved R2 49.0 mm to (36.0, 7.00), turned to 180 degrees
- moved R1 47.0 mm to (36.0, 8.45), turned to 180 degrees
- moved C1 46.2 mm to (35.0, 14.5), turned to 180 degrees
- moved C9 43.5 mm to (17.5, 11.5), turned to 180 degrees
- moved C2 42.6 mm to (35.0, 16.0), turned to 180 degrees
- moved U2 41.4 mm to (30.8, 14.9), turned to 180 degrees
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Connections:
- removed net N$1: C7.1, U3.10
- removed net N$11: C5.1, R3.2, U3.9
- removed net N$2: C15.1, U6.14
- new net MOTE_ASSOCIATED: J4.13
- new net MOTE_CONNECT: J3.6
- new net MOTE_SLEEP: J3.4
- new net MOTE_TCPSTATUS: J4.15
- net EXP_CSN: now also EXP.9; no longer J2.5
- net EXP_MISO: now also EXP.5; no longer J2.1
- net EXP_MOSI: now also EXP.8; no longer J2.4
- net EXP_SCK: now also EXP.7; no longer J2.3
- net GND: now also C4.2, EXP.10, EXP.4; no longer C13.2, C14.2, C15.2, C4.C, C5.2, C7.2, J2.6, JP4.1, JP5.1, JP6.1, JP7.1, U3.1, U3.11, U3.19, U3.8, U3.PAD, U4.3, U6.10, U6.11, U6.12, U6.13, U6.8, U6.9
- net GYRO_INT2: no longer U6.6
- net HUMID_CS: no longer U3.15
- net HUMID_VCC: no longer R3.1
- net I2C_SCL: now also EXP.2, U4.6; no longer U3.3, U4.4, U6.2
- net I2C_SDA: now also EXP.1, U4.1; no longer U3.4, U4.5, U6.3
- net LIGHT_INT: no longer U4.6
- net MOTE_ASSOC: no longer J4.15
- net MOTE_STATUS: no longer J4.13
- net VBATT: now also EXP.6; no longer C4.A, J2.2
- net VCC: now also C4.1, EXP.3, U4.5; no longer C13.1, C14.1, U4.1, U6.1, U6.15, U6.16, U6.4, U6.5
Routing:
- net GND: track 165.4 -> 0.00 mm, vias 7 -> 0
- net VCC: track 93.8 -> 0.00 mm, vias 9 -> 0
- net MOTE_SLEEPN: track 84.7 -> 0.00 mm
- net LIGHT_INT: track 72.6 -> 0.00 mm, vias 2 -> 0
- net MOTE_ASSOC: track 70.0 -> 0.00 mm, vias 2 -> 0
- net MOTE_TX_CTSN: track 67.6 -> 0.00 mm, vias 2 -> 0
- net RST: track 63.5 -> 0.00 mm, vias 2 -> 0
- net HUMID_CS: track 61.1 -> 0.00 mm, vias 2 -> 0
- net VBATT: track 59.5 -> 0.00 mm, vias 1 -> 0
- net I2C_SCL: track 58.4 -> 0.00 mm
- net I2C_SDA: track 54.9 -> 0.00 mm, vias 5 -> 0
- net ATMEGA_TO_FTDI: track 47.2 -> 0.00 mm, vias 2 -> 0
- net HUMID_VCC: track 46.6 -> 0.00 mm, vias 2 -> 0
- net MOTE_STATUS: track 46.0 -> 0.00 mm, vias 4 -> 0
- net MOTE_RESETN: track 44.9 -> 0.00 mm, vias 2 -> 0
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- removed copper zone on layer 15, net GND
- removed copper zone on layer 2, net VCC
Other:
- board outline removed
- board text removed: "U4"

Commit message: schematic and placement done?
Parts:
- removed STANDOFF4: STAND-OFF, SparkFun-Electromechanical:STAND-OFF
- added JP1, JP2: (no value), SparkFun-Connectors:1X02
- J1: device Cool_Electricity:BX0036 -> Cool_Electricity:BX0036_NOHOLES
- moved STANDOFF3 69.3 mm to (3.00, 4.00)
- moved STANDOFF1 52.0 mm to (61.0, 29.0)
- moved STANDOFF2 31.0 mm to (3.00, 29.0)
- moved R6 13.6 mm to (47.0, 20.7)
- moved C1 2.24 mm to (34.0, 12.5)
- moved C12 2.24 mm to (7.50, 15.0)
- moved C16 2.24 mm to (60.0, 14.1)
- moved C17 2.24 mm to (33.5, 21.4)
- moved C18 2.24 mm to (34.0, 29.5)
- moved C2 2.24 mm to (34.0, 14.0)
- moved C4 2.24 mm to (32.5, 24.0)
- moved C6 2.24 mm to (40.0, 17.0)
- moved C8 2.24 mm to (16.0, 24.5)
- moved C9 2.24 mm to (16.5, 9.50)
- moved EXP 2.24 mm to (47.5, 6.50)
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Connections:
- removed net GYRO_INT2: IC2.43
- removed net HUMID_CS: IC2.35
- removed net HUMID_VCC: IC2.34
- removed net MOTE_ASSOC: IC2.41
- removed net MOTE_SLEEPN: IC2.32, J3.9
- removed net MOTE_STATUS: IC2.42
- new net ADC2: IC2.35, JP2.1
- new net ADC3: IC2.34, JP2.2
- net GND: now also JP1.1, JP1.2
- net MOTE_ASSOCIATED: now also IC2.43
- net MOTE_CONNECT: now also IC2.41
- net MOTE_SLEEP: now also IC2.32
- net MOTE_TCPSTATUS: now also IC2.42
Other:
- board outline added: 63.5 x 30.5 mm

Commit message: boards submitted to fab
Parts:
- LED2: value (none) -> BLUE
- LED3: value (none) -> AMBER
- moved C1 1.50 mm to (34.0, 11.0)
- moved C10 1.50 mm to (4.50, 11.8)
- moved C11 1.50 mm to (7.50, 21.5)
- moved C12 1.50 mm to (7.50, 13.5)
- moved C16 1.50 mm to (60.0, 12.6)
- moved C17 1.50 mm to (33.5, 19.9)
- moved C18 1.50 mm to (34.0, 28.0)
- moved C2 1.50 mm to (34.0, 12.5)
- moved C3 1.50 mm to (60.0, 1.50)
- moved C4 1.50 mm to (32.5, 22.5)
- moved C6 1.50 mm to (40.0, 15.5)
- moved C8 1.50 mm to (16.0, 23.0)
- moved C9 1.50 mm to (16.5, 8.00)
- moved EXP 1.50 mm to (47.5, 5.00)
- moved IC2 1.50 mm to (17.0, 15.5)
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Routing:
- net GND: track 0.00 -> 230.2 mm, vias 0 -> 5
- net VCC: track 0.00 -> 190.5 mm, vias 0 -> 4
- net VBATT: track 0.00 -> 108.2 mm, vias 0 -> 1
- net I2C_SDA: track 0.00 -> 82.7 mm, vias 0 -> 4
- net LIGHT_INT: track 0.00 -> 80.9 mm, vias 0 -> 2
- net RST: track 0.00 -> 80.2 mm, vias 0 -> 5
- net I2C_SCL: track 0.00 -> 67.9 mm, vias 0 -> 7
- net TCK: track 0.00 -> 49.8 mm, vias 0 -> 1
- net TDO: track 0.00 -> 47.7 mm, vias 0 -> 2
- net PIR_VCC: track 0.00 -> 46.8 mm, vias 0 -> 3
- net MOTE_CONNECT: track 0.00 -> 46.2 mm, vias 0 -> 4
- net LED1: track 0.00 -> 46.2 mm, vias 0 -> 2
- net PIR_OUT: track 0.00 -> 46.0 mm, vias 0 -> 2
- net LED2: track 0.00 -> 44.6 mm, vias 0 -> 2
- net TMS: track 0.00 -> 44.6 mm, vias 0 -> 3
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- added copper zone on layer 1, net GND
- added copper zone on layer 16, net GND
Other:
- board text added: "JTAG"

Commit message: Updated board design and shipping
Parts:
- removed R5: 0R DNP, resistor:R0603
- added POW: POWER, Cool_Electricity:JS102011SAQN
- EXP: value M05X2SHD -> M05X2SHD_SMD; device SparkFun-Connectors:2X5-SHROUDED -> SparkFun-Connectors:2X5-SHROUDED_SMD
- JP9: device SparkFun-Connectors:2X5-SHROUDED -> SparkFun-Connectors:2X5-SHROUDED_SMD
- moved C16 2.06 mm to (62.0, 13.1)
- moved C3 2.06 mm to (62.0, 2.00)
- moved LED2 2.06 mm to (62.0, 10.8)
- moved LED3 2.06 mm to (62.0, 8.50)
- moved U1 2.06 mm to (62.0, 5.10)
- moved STANDOFF1 1.50 mm to (61.0, 29.0)
- moved EXP 0.71 mm to (48.0, 5.50)
- moved J3 0.71 mm to (21.0, 16.0)
- moved J4 0.71 mm to (21.0, 16.0)
- moved JP9 0.71 mm to (48.0, 26.5)
- moved C1 0.50 mm to (34.0, 11.5)
- moved C10 0.50 mm to (4.50, 12.3)
- moved C11 0.50 mm to (7.50, 22.0)
- moved C12 0.50 mm to (7.50, 14.0)
- moved C17 0.50 mm to (33.5, 20.4)
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Connections:
- new net N$1: J1.POS, POW.1
- net VBATT: now also POW.C; no longer J1.POS, R5.2
- net VCC: no longer R5.1
Routing:
- net GND: track 230.2 -> 189.7 mm, vias 5 -> 68
- net MOTE_CONNECT: track 46.2 -> 19.8 mm
- net VBATT: track 108.2 -> 84.9 mm, vias 1 -> 3
- net PIR_VCC: track 46.8 -> 69.2 mm, vias 3 -> 5
- net LIGHT_INT: track 80.9 -> 59.6 mm, vias 2 -> 4
- net RST: track 80.2 -> 60.8 mm, vias 5 -> 7
- net I2C_SDA: track 82.7 -> 68.1 mm, vias 4 -> 6
- net ATMEGA_TO_FTDI: track 42.5 -> 31.7 mm, vias 1 -> 2
- net MOTE_RX_RTSN: track 28.9 -> 19.2 mm, vias 2 -> 4
- net LED1: track 46.2 -> 54.5 mm
- net VCC: track 190.5 -> 183.4 mm, vias 4 -> 5
- net TCK: track 49.8 -> 43.3 mm, vias 1 -> 2
- net ACCEL_INT2: track 21.5 -> 15.9 mm
- net MOTE_TX_CTSN: track 7.77 -> 13.3 mm
- net TMS: track 44.6 -> 39.3 mm, vias 3 -> 2
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Other:
- board size 63.5 x 30.5 mm -> 64.5 x 32 mm
- board text added: "ESENSE v3.1 Kevin Weekly"
- board text removed: "Environmental Sensor PCB Kevin Weekly"
